File: pcb/mem_pmod/mem_pmod.kicad_sch (KiCad schematic)
At the start: 14 parts, among them J1 Conn_01x04_Pin, U1 74HC125D

Commit message: Replacing components in schematic due to prop delay
Parts:
- removed Demux: 74ACT139MTCX, TSSOP16_5X4P5_ONS, symbol demux:74ACT139MTCX
- removed NOT: SN74HCS14DYYR, SOP50P326X110-14N, symbol SN74HCS14DYYR:SN74HCS14DYYR
Connections:
- no-connect marks 2 -> 0
Other:
- moved on the sheet: Flash, RAM0, RAM1, RAM2
